Commit message: update

File: resources/robots/h1_2/h1_2_simplified.urdf (robot description, URDF)
Before this commit: robot h1_5, 56 links, 55 joints
Links:
- link L_hand_base_link: geometry collision mesh filename=meshes/L_hand_base_link.STL; visual mesh filename=meshes/L_hand_base_link.STL
- link R_hand_base_link: geometry collision mesh filename=meshes/R_hand_base_link.STL; visual mesh filename=meshes/R_hand_base_link.STL
- link left_ankle_roll_link: geometry collision mesh filename=meshes/left_ankle_roll_link.STL; visual mesh filename=meshes/left_ankle_roll_link.STL
- link left_elbow_roll_link: geometry collision mesh filename=meshes/left_elbow_roll_link.STL; visual mesh filename=meshes/left_elbow_roll_link.STL
- link left_hip_roll_link: geometry collision cylinder length=0.01 radius=0.02; visual mesh filename=meshes/left_hip_roll_link.STL
- link right_ankle_roll_link: geometry collision mesh filename=meshes/right_ankle_roll_link.STL; visual mesh filename=meshes/right_ankle_roll_link.STL
- link right_elbow_roll_link: geometry collision mesh filename=meshes/right_elbow_roll_link.STL; visual mesh filename=meshes/right_elbow_roll_link.STL
- link right_hip_roll_link: geometry collision cylinder length=0.01 radius=0.02; visual mesh filename=meshes/right_hip_roll_link.STL

Commit message: add height termination

File: resources/robots/h1_2/h1_2_simplified.urdf (robot description, URDF)
Before this commit: robot h1_5, 56 links, 55 joints
Links:
- link left_hip_pitch_link: geometry collision cylinder length=0.2 radius=0.02; visual mesh filename=meshes/left_hip_pitch_link.STL
- link left_hip_yaw_link: geometry collision cylinder length=0.02 radius=0.01; visual mesh filename=meshes/left_hip_yaw_link.STL
- link left_shoulder_pitch_link: geometry collision mesh filename=meshes/left_shoulder_pitch_link.STL; visual mesh filename=meshes/left_shoulder_pitch_link.STL
- link right_hip_pitch_link: geometry collision cylinder length=0.2 radius=0.02; visual mesh filename=meshes/right_hip_pitch_link.STL
- link right_hip_yaw_link: geometry collision cylinder length=0.02 radius=0.01; visual mesh filename=meshes/right_hip_yaw_link.STL
- link right_shoulder_pitch_link: geometry collision mesh filename=meshes/right_shoulder_pitch_link.STL; visual mesh filename=meshes/right_shoulder_pitch_link.STL
